File: Yudao.sch (KiCad schematic (older format))
At the start: 5 parts, among them Q1 BC548

Commit message: Selecionar footprints
Footprints selecionadas
Parts:
- C1: footprint (none) -> Capacitor_THT:C_Disc_D3.4mm_W2.1mm_P2.50mm
- R1, R2, R3: footprint (none) -> Resistor_THT:R_Axial_DIN0207_L6.3mm_D2.5mm_P7.62mm_Horizontal
Changed lines of the file:
@@
 F 0 "R1" V 1846 4050 50  0000 C CNN
 F 1 "1k" V 1755 4050 50  0000 C CNN
-F 2 "" H 1650 4050 50  0001 C CNN
+F 2 "Resistor_THT:R_Axial_DIN0207_L6.3mm_D2.5mm_P7.62mm_Horizontal" H 1650 4050 50  0001 C CNN
 F 3 "~" H 1650 4050 50  0001 C CNN
 	1    1650 4050
@@
 F 0 "R3" H 1941 4354 50  0000 R CNN
 F 1 "510k" H 1941 4445 50  0000 R CNN
-F 2 "" H 2000 4400 50  0001 C CNN
+F 2 "Resistor_THT:R_Axial_DIN0207_L6.3mm_D2.5mm_P7.62mm_Horizontal" H 2000 4400 50  0001 C CNN
 F 3 "~" H 2000 4400 50  0001 C CNN
 	1    2000 4400
@@
 F 0 "C1" V 1121 4050 50  0000 C CNN
 F 1 "20nF" V 1212 4050 50  0000 C CNN
-F 2 "" H 1350 4050 50  0001 C CNN
+F 2 "Capacitor_THT:C_Disc_D3.4mm_W2.1mm_P2.50mm" H 1350 4050 50  0001 C CNN
 F 3 "~" H 1350 4050 50  0001 C CNN
 	1    1350 4050
@@
 F 0 "R2" H 2491 4504 50  0000 R CNN
 F 1 "10k" H 2491 4595 50  0000 R CNN
-F 2 "" H 2550 4550 50  0001 C CNN
+F 2 "Resistor_THT:R_Axial_DIN0207_L6.3mm_D2.5mm_P7.62mm_Horizontal" H 2550 4550 50  0001 C CNN
 F 3 "~" H 2550 4550 50  0001 C CNN
 	1    2550 4550
@@
 $EndComp
 $Comp
-L power:GND #PWR?
+L power:GND #PWR01
 U 1 1 5D4E5500
 P 2000 4650
-F 0 "#PWR?" H 2000 4400 50  0001 C CNN
+F 0 "#PWR01" H 2000 4400 50  0001 C CNN
 F 1 "GND" H 2005 4477 50  0000 C CNN
 F 2 "" H 2000 4650 50  0001 C CNN
@@
 $EndComp
 $Comp
-L power:VCC #PWR?
+L power:VCC #PWR02
 U 1 1 5D4E5973
 P 2550 3750
-F 0 "#PWR?" H 2550 3600 50  0001 C CNN
+F 0 "#PWR02" H 2550 3600 50  0001 C CNN
 F 1 "VCC" H 2567 3923 50  0000 C CNN
 F 2 "" H 2550 3750 50  0001 C CNN
@@
 	2550 3850 2550 3750
 $Comp
-L power:GND #PWR?
+L power:GND #PWR03
 U 1 1 5D4EB89E
 P 2550 4750
-F 0 "#PWR?" H 2550 4500 50  0001 C CNN
+F 0 "#PWR03" H 2550 4500 50  0001 C CNN
 F 1 "GND" H 2555 4577 50  0000 C CNN
 F 2 "" H 2550 4750 50  0001 C CNN
